File: schematics/PSLab.kicad_sch (KiCad schematic)
At the start: 198 parts, among them J1 DoublePins, J10 Programmer, J11 Battery_Cell, J12 USB_C_Receptacle, J13 CR1225, J2 Conn_01x25, J3 Conn_01x13, J6 ESP01, J8 Micro_SD_Card_Det_9_pin, Q1 MMBT3906, Q2 MMBT3904, Q3 MMBT3906, SW1 SW_MEC_5E, SW2 SW_MEC_5E, SW3 SW_MEC_5E, U1 AP3015A, U10 TL082, U11 TL082, U12 74HC4051, U13 TL082, U14 MCP6S21, U15 CP2102N-xxx-xQFN20x, U16 SP0503BAHT, U17 MT1470, U18 MCP6S21, U2 74HC126, U20 MCP4822, U21 IP5189T, U3 PIC24EP256GP204, U4 DS1307Z+T&R, U6 AMS1117-3.3, U7 LM324, U9 TL082, X1 12MHz, X2 32.768 kHz

Commit message: feat: PSLab Mini prototype v1.0
Parts:
- removed C1, C2, C24, C27, C32, C34, C35, C37, C38, C9: 100nF, Capacitor_SMD:C_0603_1608Metric, symbol Device:C
- removed C11: 2.2uF, Capacitor_SMD:C_0603_1608Metric, symbol Device:C_Small
- removed C12, C14: 10uF, Capacitor_SMD:C_0603_1608Metric, symbol Device:C_Small
- removed C15, C33, C6: 10uF, Capacitor_SMD:C_0603_1608Metric, symbol Device:C
- removed C18: 100nF, Capacitor_SMD:C_0603_1608Metric, symbol Device:C_Small
- removed C20, C42: 1uF, Capacitor_SMD:C_0603_1608Metric, symbol Device:C
- removed C30, C36: 1nF, Capacitor_SMD:C_0603_1608Metric, symbol Device:C
- removed C40, C7: 10nF, Capacitor_SMD:C_0603_1608Metric, symbol Device:C
- removed C45, C46, C47, C48, C49, C50, C51, C54: 22uF, Capacitor_SMD:C_0603_1608Metric, symbol Device:C_Small
- removed C52: 1uF, Capacitor_SMD:C_0603_1608Metric, symbol Device:C_Small
- removed C53: 12pF, Capacitor_SMD:C_0603_1608Metric, symbol Device:C_Small
- removed D1: 6.8V, Diode_SMD:D_MiniMELF, symbol Device:D_Zener_Small_Filled
- removed D10, D11, D12, D13: White, LED_SMD:LED_0603_1608Metric, symbol Device:LED_Small
- removed D7: K1N5817HW-7-F, Diode_SMD:D_SOD-123, symbol Device:D_Schottky
- removed D8: 1N4148W, Diode_SMD:D_MiniMELF, symbol Device:D
- removed J11: Battery_Cell, PSLab:2.0mm_connector_edge, symbol Device:Battery_Cell
- removed J13: CR1225, PSLab:BatteryHolder_A359, symbol Device:Battery_Cell
- removed J2: Conn_01x25, Connector_PinSocket_2.54mm:PinSocket_1x25_P2.54mm_Vertical, symbol Connector_Generic:Conn_01x25
- removed J3: Conn_01x13, Connector_PinSocket_2.54mm:PinSocket_1x13_P2.54mm_Vertical, symbol Connector_Generic:Conn_01x13
- removed J6: ESP01, PSLab:ESP-01, symbol PSLab:ESP01
- removed J8: Micro_SD_Card_Det_9_pin, PSLab:TF-015, symbol PSLab:Micro_SD_Card_Det_9_pin
- removed L1: 3.3uH, Inductor_SMD:L_Taiyo-Yuden_MD-2020, symbol Device:L
- removed L2: 4.7uH, Inductor_SMD:L_Taiyo-Yuden_MD-2020, symbol Device:L_Small
- removed L3, L4: 3.3uH, Inductor_SMD:L_Taiyo-Yuden_MD-2020, symbol Device:L_Small
- removed Q1: MMBT3906, Package_TO_SOT_SMD:SOT-23, symbol Transistor_BJT:MMBT3906
- removed Q2: MMBT3904, Package_TO_SOT_SMD:SOT-23, symbol Device:Q_NPN_BEC
- removed R13, R27, R28, R62: 200, Resistor_SMD:R_0603_1608Metric, symbol Device:R_Small
- removed R14, R18, R19, R21, R25, R31, R32, R33, R35, R37, R38, R39, R42: 10k, Resistor_SMD:R_0603_1608Metric, symbol Device:R
- removed R15, R26, R41, R43, R44: 5.1k, Resistor_SMD:R_0603_1608Metric, symbol Device:R
- removed R36, R47, R5: 1k, Resistor_SMD:R_0603_1608Metric, symbol Device:R
- removed R40, R46, R50: 200k, Resistor_SMD:R_0603_1608Metric, symbol Device:R
- removed R45: 1M, Resistor_SMD:R_0603_1608Metric, symbol Device:R
- removed R61: 51k, Resistor_SMD:R_0603_1608Metric, symbol Device:R_Small
- removed R63, R77: 200k, Resistor_SMD:R_0603_1608Metric, symbol Device:R_Small
- removed R68: 180k, Resistor_SMD:R_0603_1608Metric, symbol Device:R_Small
- removed R69: 30k, Resistor_SMD:R_0603_1608Metric, symbol Device:R_Small
- removed R70, R76: 10k, Resistor_SMD:R_0603_1608Metric, symbol Device:R_Small
- removed R75: 100k, Resistor_SMD:R_0603_1608Metric, symbol Device:R_Small
- removed SW3: SW_MEC_5E, PSLab:button_SPST_3x4x2.5, symbol Switch:SW_MEC_5E
- removed U1: AP3015A, Package_TO_SOT_SMD:SOT-23-5, symbol PSLab:AP3015A
- removed U10, U11: TL082, Package_SO:SOIC-8_3.9x4.9mm_P1.27mm, symbol Amplifier_Operational:TL082
- removed U17: MT1470, Package_TO_SOT_SMD:SOT-23-6, symbol PSLab:MT1470
- removed U2: 74HC126, Package_SO:TSSOP-14_4.4x5mm_P0.65mm, symbol 74xx:74LS126
- removed U20: MCP4822, Package_SO:SOIC-8_3.9x4.9mm_P1.27mm, symbol Analog_DAC:MCP4822
- removed U21: IP5189T, Package_DFN_QFN:QFN-24-1EP_4x4mm_P0.5mm_EP2.6x2.6mm, symbol PSLab:IP5189T
- removed U4: DS1307Z+T&R, Package_SO:SOIC-8_3.9x4.9mm_P1.27mm, symbol Timer_RTC:DS1307Z+
- removed U6: AMS1117-3.3, Package_TO_SOT_SMD:SOT-223-3_TabPin2, symbol Regulator_Linear:AMS1117-3.3
- removed U7: LM324, Package_SO:TSSOP-14_4.4x5mm_P0.65mm, symbol Amplifier_Operational:LM324
- removed X2: 32.768 kHz, Crystal:Crystal_SMD_3215-2Pin_3.2x1.5mm, symbol Device:Crystal_Small
- removed Z1: CR1225, Battery:Battery_CR1225, symbol PSLab:Battery
- added SPI_Socket1: Conn_01x06, symbol Connector_Generic:Conn_01x06
- added UART_Socket1: Conn_01x04, symbol Connector_Generic:Conn_01x04
Connections:
- net +3.3V: now also SPI_Socket1.6 (Pin_6)
- net +5V: now also UART_Socket1.1 (Pin_1)
- net GND: now also SPI_Socket1.5 (Pin_5), UART_Socket1.2 (Pin_2)
- net RxD2: now also UART_Socket1.4 (Pin_4)
- net SCK: now also SPI_Socket1.3 (Pin_3)
- net SDI: now also SPI_Socket1.2 (Pin_2)
- net SDO: now also SPI_Socket1.4 (Pin_4)
- net SPI.CS: now also SPI_Socket1.1 (Pin_1)
- net TxD2: now also UART_Socket1.3 (Pin_3)
- net CH3: no longer names the net of J1.14 (Pin_14)
- net CH3.GAIN: no longer names the net of J1.12 (Pin_12)
- net CH3_IN: no longer names the net of U3.20 (AN1|C2IN1+|RA1)
- net MIC: no longer names the net of J1.10 (Pin_10)
- net MIC_IN: no longer names the net of U3.21 (PGED3|AN2|C2IN1-|RPI32|RB0)
- net SD.CS: no longer names the net of R72.1, U12.5 (A5)
- no-connect marks 32 -> 16
Other:
- note added: "05"
- note added: "06"
- note added: "07"
- note added: "08"
- note added: "09"
- note added: "10"
- note added: "11"
- note added: "12"
- note added: "13"
- note added: "14"
- note added: "15"
- note added: "16"
- note added: "17"
- note added: "18"
- note added: "19"
- note added: "21"
- note added: "22"
- note added: "23"
- note added: "24"
- note added: "25"
- note added: "26"
- note added: "3 oscilloscope channels not required"
- note added: "A Real Time Clock Module is not necessary in PSLab Mini"
- note added: "ESP Integration not necessary"
- note added: "Needed for oscilloscope"
- note added: "No Audio Channel required"
- note added: "No Power Source module in pslab mini"
- note added: "No Sine Wave Generator in PSLab Mini"
- note added: "SD Card is redundant in PSLab Data Stored digitally"
- note added: "These not required ,as no power supply module"
- note removed: "Audio Channel"
- note removed: "Battery Backup System"
- note removed: "ESP-01 Expansion Slot"
- note removed: "I_chg = 100k * 1.2V / R_chg = 0.6A"
- note removed: "Oscilloscope Channel 03"
- note removed: "Power Source"
- note removed: "Real Time Clock Module"
- note removed: "Sine Wave Generator"
- note removed: "Voltage Doubler"
- note removed: "Voltage Inverter Regulator"
- note removed: "Vout=0.8*110k/10k=8.8V"
- note removed: "Vout=1.23*210k/30k=8.61V"
- title: PSLab Board Schematic -> PSLab Mini Board Schematic
- moved on the sheet: J1, J10
